File: hardware/kicad_magsafe_dock/openmotorbridge_magsafe_dock.kicad_sch (KiCad schematic)
At the start: 6 parts, among them J1 M8_6PIN_CABLE_PADS, J2 MAGSAFE_6PIN_RECEPTACLE, U1 USBLC6-4SC6

Commit message: feat(cad/pcb): redesign PCBA 06 and MagSafe frame dock enclosure with horizontal clamshell & central M2.5 boss
Connections:
- net at J1.4 (4_SIG_N): now also U1.6 (IO4); no longer U1.3 (IO2)
- net at J1.5 (5_TRIGGER_PPS): now also U1.3 (IO2); no longer U1.4 (IO3)
- net at J1.6 (6_1WIRE_ID): now also U1.4 (IO3); no longer U1.6 (IO4)
Changed lines of the file:
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@@
 	(wire (pts (xy 37.38 57.46) (xy 74.84 76.19)) (stroke (width 0) (type solid)))
 	(wire (pts (xy 74.84 76.19) (xy 127.38 58.73)) (stroke (width 0) (type solid)))
-	(wire (pts (xy 37.38 60.0) (xy 74.84 83.81)) (stroke (width 0) (type solid)))
-	(wire (pts (xy 74.84 83.81) (xy 127.38 61.27)) (stroke (width 0) (type solid)))
-	(wire (pts (xy 37.38 62.54) (xy 95.16 83.81)) (stroke (width 0) (type solid)))
-	(wire (pts (xy 95.16 83.81) (xy 127.38 63.81)) (stroke (width 0) (type solid)))
-	(wire (pts (xy 37.38 65.08) (xy 95.16 76.19)) (stroke (width 0) (type solid)))
-	(wire (pts (xy 95.16 76.19) (xy 127.38 66.35)) (stroke (width 0) (type solid)))
+	(wire (pts (xy 37.38 60.0) (xy 95.16 76.19)) (stroke (width 0) (type solid)))
+	(wire (pts (xy 95.16 76.19) (xy 127.38 61.27)) (stroke (width 0) (type solid)))
+	(wire (pts (xy 37.38 62.54) (xy 74.84 83.81)) (stroke (width 0) (type solid)))
+	(wire (pts (xy 74.84 83.81) (xy 127.38 63.81)) (stroke (width 0) (type solid)))
+	(wire (pts (xy 37.38 65.08) (xy 95.16 83.81)) (stroke (width 0) (type solid)))
+	(wire (pts (xy 95.16 83.81) (xy 127.38 66.35)) (stroke (width 0) (type solid)))
 )
