File: hardware/kicad_main_box/power_supply_ups.kicad_sch (KiCad schematic)
At the start: 6 parts, among them U1 LM5164-Q1, U7 TPS7A0533

Commit message: hardware(schematic): assign exact footprints to all hierarchical schematic symbols
- Assign SMD footprints for ESP32-S3, ES8388, TCAN334G, LM5164-Q1, TPS7A0533
- Assign footprints for Bourns LM-NP-1001 transformers, TLP222A PhotoMOS, TVS, passives, and IDC26 connector
- Fix F8 PCB netlist synchronization (0 unassigned footprint errors)
Parts:
- C1, C2: footprint (none) -> Capacitor_SMD:C_0805_2012Metric
- D1: footprint (none) -> Diode_SMD:D_SMB
- L1: footprint (none) -> Inductor_SMD:L_2816_7142Metric
- U1: footprint (none) -> Package_SO:SOIC-8-1EP_3.9x4.9mm_P1.27mm_EP2.41x3.3mm
- U7: footprint (none) -> Package_TO_SOT_SMD:SOT-23-5
Changed lines of the file:
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@@
 		(property "Reference" "D1" (at 48.0 58.0 0) (effects (font (size 1.27 1.27))))
 		(property "Value" "SMBJ36A" (at 48.0 62.0 0) (effects (font (size 1.27 1.27))))
+		(property "Footprint" "Diode_SMD:D_SMB" (at 0 0 0) (effects (font (size 1.27 1.27)) (hide yes)))
 		(pin "1")
 		(pin "2")
@@
 		(property "Reference" "C1" (at 63.0 58.0 0) (effects (font (size 1.27 1.27))))
 		(property "Value" "100uF/50V" (at 63.0 62.0 0) (effects (font (size 1.27 1.27))))
+		(property "Footprint" "Capacitor_SMD:C_0805_2012Metric" (at 0 0 0) (effects (font (size 1.27 1.27)) (hide yes)))
 		(pin "1")
 		(pin "2")
@@
 		(property "Reference" "U1" (at 100.0 48.0 0) (effects (font (size 1.27 1.27))))
 		(property "Value" "LM5164-Q1" (at 100.0 51.0 0) (effects (font (size 1.27 1.27))))
+		(property "Footprint" "Package_SO:SOIC-8-1EP_3.9x4.9mm_P1.27mm_EP2.41x3.3mm" (at 0 0 0) (effects (font (size 1.27 1.27)) (hide yes)))
 		(pin "1")
 		(pin "2")
@@
 		(property "Reference" "L1" (at 130.0 50.0 0) (effects (font (size 1.27 1.27))))
 		(property "Value" "47uH" (at 130.0 53.0 0) (effects (font (size 1.27 1.27))))
+		(property "Footprint" "Inductor_SMD:L_2816_7142Metric" (at 0 0 0) (effects (font (size 1.27 1.27)) (hide yes)))
 		(pin "1")
 		(pin "2")
@@
 		(property "Reference" "C2" (at 153.0 58.0 0) (effects (font (size 1.27 1.27))))
 		(property "Value" "10uF/16V" (at 153.0 62.0 0) (effects (font (size 1.27 1.27))))
+		(property "Footprint" "Capacitor_SMD:C_0805_2012Metric" (at 0 0 0) (effects (font (size 1.27 1.27)) (hide yes)))
 		(pin "1")
 		(pin "2")
@@
 		(property "Reference" "U7" (at 185.0 60.0 0) (effects (font (size 1.27 1.27))))
 		(property "Value" "TPS7A0533" (at 185.0 63.0 0) (effects (font (size 1.27 1.27))))
+		(property "Footprint" "Package_TO_SOT_SMD:SOT-23-5" (at 0 0 0) (effects (font (size 1.27 1.27)) (hide yes)))
 		(pin "1")
 		(pin "2")

Commit message: hardware(pcb): fix official KiCad library footprint names for U3 and L1
- Update U3 to official KiCad footprint Package_DFN_QFN:QFN-28-1EP_4x4mm_P0.4mm_EP2.4x2.4mm
- Update L1 to official KiCad footprint Inductor_SMD:L_Sunlord_MWSA1206S-470
- Complete 100% F8 schematic-to-PCB synchronization with 0 errors
Parts:
- L1: footprint Inductor_SMD:L_2816_7142Metric -> Inductor_SMD:L_Sunlord_MWSA1206S-470
Changed lines of the file:
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@@
 		(property "Reference" "L1" (at 130.0 50.0 0) (effects (font (size 1.27 1.27))))
 		(property "Value" "47uH" (at 130.0 53.0 0) (effects (font (size 1.27 1.27))))
-		(property "Footprint" "Inductor_SMD:L_2816_7142Metric" (at 0 0 0) (effects (font (size 1.27 1.27)) (hide yes)))
+		(property "Footprint" "Inductor_SMD:L_Sunlord_MWSA1206S-470" (at 0 0 0) (effects (font (size 1.27 1.27)) (hide yes)))
 		(pin "1")
 		(pin "2")

Commit message: hardware(schematic): align schematic reference designators with PCB layout
- Rename Q1 -> U7 in audio_frontend_isolated (TLP222A Opto1)
- Rename U7 -> U9 in power_supply_ups (TPS7A0533 LDO)
- Rename D1 -> D2 in power_supply_ups (SMBJ33CA TVS)
- Fix 100% 1:1 symbol-to-PCB reference mapping (0 unplaced ghost components on mouse cursor)
Parts:
- renumbered D1 to D2, U7 to U9
Changed lines of the file:
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@@
 	(symbol (lib_id "Device:D_TVS") (at 45.0 60.0 0) (unit 1)
 		(in_bom yes) (on_board yes) (dnp no)
-		(property "Reference" "D1" (at 48.0 58.0 0) (effects (font (size 1.27 1.27))))
+		(property "Reference" "D2" (at 48.0 58.0 0) (effects (font (size 1.27 1.27))))
 		(property "Value" "SMBJ36A" (at 48.0 62.0 0) (effects (font (size 1.27 1.27))))
 		(property "Footprint" "Diode_SMD:D_SMB" (at 0 0 0) (effects (font (size 1.27 1.27)) (hide yes)))
@@
 	(symbol (lib_id "Regulator_Linear:TPS7A0533") (at 185.0 70.0 0) (unit 1)
 		(in_bom yes) (on_board yes) (dnp no)
-		(property "Reference" "U7" (at 185.0 60.0 0) (effects (font (size 1.27 1.27))))
+		(property "Reference" "U9" (at 185.0 60.0 0) (effects (font (size 1.27 1.27))))
 		(property "Value" "TPS7A0533" (at 185.0 63.0 0) (effects (font (size 1.27 1.27))))
 		(property "Footprint" "Package_TO_SOT_SMD:SOT-23-5" (at 0 0 0) (effects (font (size 1.27 1.27)) (hide yes)))

Commit message: fix(main_box): clean up schematics, connect LoRa/UWB/IMU/SD/LED nets, verify J2 MicroSD placement
Parts:
- renumbered U9 to U11
Changed lines of the file:
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@@
 		(in_pos_files yes)
 		(dnp no)
-		(property "Reference" "U9"
+		(property "Reference" "U11"
 			(at 185 60 0)
 			(show_name no)
@@
 			(project "openmotorbridge_main"
 				(path "/a0000000-0000-0000-0000-000000000001/a0000000-0000-0000-0000-000000000002"
-					(reference "U9")
+					(reference "U11")
 					(unit 1)
 				)
