File: hardware/kicad_main_box/dtm12_interface.kicad_sch (KiCad schematic)
At the start: 1 part, among them J1 DEUTSCH_DTM12_IDC_HEADER

Commit message: fix(hardware): fleet-wide 7-PCBA remediation, schematic parity & doc alignment
- PCBA 01 (Central Box): Synchronized DTM-12 schematic and PCB routing, purged obsolete analog audio transformers/HD26 connector.
- PCBA 03 (Smart Cartridge): Verified Kelvin ground isolation on J_AUDIO_PWR, resolved U1.16 BAY_SELECT single net.
- PCBA 05 (Front Node): Mapped DW3110 UWB SPI/IRQ/RST to ESP32-S3 pads 30-35, connected MK1 I2S MEMS mic and Y_UWB crystal.
- PCBA 07 (Smart Keyfob): Connected 12 unrouted signals (SX1262 LoRa SPI, DRV2605L I2C, SWD, RTC crystal, buttons) to nRF52840 pads.
- PCBA 08 (Radar Sub-MCU): Synchronized J1.1 power rail to VCC_5V, connected Y1_UWB crystal to DW3110 pads 4 & 5.
- PCBA 09 & PCBA 10 (OMM 2.4 GHz & 446 MHz): Verified 4-layer stackup, BQ24075 ground ties, SA818 isolation, and vertical B.Cu J_HELMET orientation.
- Tools: Added verify_hardware_integrity.py with automated DRC/parity/single-net/floating-pad checks (all 7 PCBAs HEALTHY).
- Docs: Synchronized docs/de and docs/en hardware specifications, pinouts, and DTM-12 architecture.
Connections:
- net CAN_H: now also J1.8
- net CAN_L: now also J1.5
- net GND_PWR: now also J1.1, J1.3, J1.7
- net KL15_IGN: now also J1.10
- net KL30_IN: now also J1.9
- net POD1_VCC: now also J1.6
- net POD2_VCC: now also J1.4
- net RADAR_PWR_12V: now also J1.2
Changed lines of the file:
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@@
 	(title_block
 		(title "OpenMotorBridge v9.6 - Deutsch DTM-12 Interface")
-		(date "2026-10-09")
+		(date "2026-10-14")
 		(rev "v9.6")
 		(company "OpenMotorBridge Open Source Hardware")
@@
 		(pin "12")
 	)
+	(wire (pts (xy 52.07 71.12) (xy 30.48 71.12)) (stroke (width 0) (type default)) (uuid "w1000000-0000-0000-0000-000000000001"))
+	(wire (pts (xy 69.85 71.12) (xy 88.90 71.12)) (stroke (width 0) (type default)) (uuid "w1000000-0000-0000-0000-000000000002"))
+	(wire (pts (xy 52.07 66.04) (xy 30.48 66.04)) (stroke (width 0) (type default)) (uuid "w1000000-0000-0000-0000-000000000003"))
+	(wire (pts (xy 69.85 66.04) (xy 88.90 66.04)) (stroke (width 0) (type default)) (uuid "w1000000-0000-0000-0000-000000000004"))
+	(wire (pts (xy 52.07 60.96) (xy 30.48 60.96)) (stroke (width 0) (type default)) (uuid "w1000000-0000-0000-0000-000000000005"))
+	(wire (pts (xy 69.85 60.96) (xy 88.90 60.96)) (stroke (width 0) (type default)) (uuid "w1000000-0000-0000-0000-000000000006"))
+	(wire (pts (xy 52.07 55.88) (xy 30.48 55.88)) (stroke (width 0) (type default)) (uuid "w1000000-0000-0000-0000-000000000007"))
+	(wire (pts (xy 69.85 55.88) (xy 88.90 55.88)) (stroke (width 0) (type default)) (uuid "w1000000-0000-0000-0000-000000000008"))
+	(wire (pts (xy 52.07 50.80) (xy 30.48 50.80)) (stroke (width 0) (type default)) (uuid "w1000000-0000-0000-0000-000000000009"))
+	(wire (pts (xy 69.85 50.80) (xy 88.90 50.80)) (stroke (width 0) (type default)) (uuid "w1000000-0000-0000-0000-00000000000A"))
+	(wire (pts (xy 52.07 45.72) (xy 30.48 45.72)) (stroke (width 0) (type default)) (uuid "w1000000-0000-0000-0000-00000000000B"))
+	(wire (pts (xy 69.85 45.72) (xy 88.90 45.72)) (stroke (width 0) (type default)) (uuid "w1000000-0000-0000-0000-00000000000C"))
 	(hierarchical_label "KL30_IN" (shape output) (at 30.48 71.12 180) (effects (font (size 1.27 1.27)) (justify right)))
-	(hierarchical_label "KL15_IGN" (shape output) (at 88.9 71.12 0) (effects (font (size 1.27 1.27)) (justify left)))
+	(hierarchical_label "KL15_IGN" (shape output) (at 88.90 71.12 0) (effects (font (size 1.27 1.27)) (justify left)))
 	(hierarchical_label "GND_PWR" (shape output) (at 30.48 66.04 180) (effects (font (size 1.27 1.27)) (justify right)))
-	(hierarchical_label "CAN_H" (shape bidirectional) (at 88.9 66.04 0) (effects (font (size 1.27 1.27)) (justify left)))
+	(hierarchical_label "CAN_H" (shape bidirectional) (at 88.90 66.04 0) (effects (font (size 1.27 1.27)) (justify left)))
 	(hierarchical_label "CAN_L" (shape bidirectional) (at 30.48 60.96 180) (effects (font (size 1.27 1.27)) (justify right)))
-	(hierarchical_label "POD1_VCC" (shape input) (at 88.9 60.96 0) (effects (font (size 1.27 1.27)) (justify left)))
-	(hierarchical_label "POD2_VCC" (shape input) (at 88.9 50.8 0) (effects (font (size 1.27 1.27)) (justify left)))
-	(hierarchical_label "RADAR_PWR_12V" (shape input) (at 88.9 45.72 0) (effects (font (size 1.27 1.27)) (justify left)))
-	(hierarchical_label "CHASSIS_EARTH" (shape passive) (at 88.9 40.64 0) (effects (font (size 1.27 1.27)) (justify left)))
+	(hierarchical_label "POD1_VCC" (shape input) (at 88.90 60.96 0) (effects (font (size 1.27 1.27)) (justify left)))
+	(hierarchical_label "GND_PWR" (shape output) (at 30.48 55.88 180) (effects (font (size 1.27 1.27)) (justify right)))
+	(hierarchical_label "POD2_VCC" (shape input) (at 88.90 55.88 0) (effects (font (size 1.27 1.27)) (justify left)))
+	(hierarchical_label "GND_PWR" (shape output) (at 30.48 50.80 180) (effects (font (size 1.27 1.27)) (justify right)))
+	(hierarchical_label "RADAR_PWR_12V" (shape input) (at 88.90 50.80 0) (effects (font (size 1.27 1.27)) (justify left)))
+	(hierarchical_label "GND_PWR" (shape output) (at 30.48 45.72 180) (effects (font (size 1.27 1.27)) (justify right)))
+	(hierarchical_label "CHASSIS_EARTH" (shape passive) (at 88.90 45.72 0) (effects (font (size 1.27 1.27)) (justify left)))
 )
