File: hardware/kicad_main_box/openmotorbridge_main.kicad_sch (KiCad schematic)
At the start: 37 parts, among them J1 DEUTSCH_DTM12_IDC_HEADER, J2 MicroSD_Card, J3 USB2_IDC_HEADER_9PIN, J4 RGB_LED_3PIN, J5 PWR_BAT_NTC_4PIN, SW1 SW_PAIR_RESET, U1 LM5164-Q1, U10 SX1262IMLTRT, U11 TPS7A0533_LDO, U2 ESP32-S3-WROOM-1U-N16R8, U3 ES8388_Codec, U5 BMI270_IMU, U6 TCAN334G, U8 DW3110, U9 QCC3084_BT54_AUDIO, Y1_UWB 38.4MHz

Commit message: hw(pcba): synchronize schematic-to-pcb parity and update central box v10 layout
- Synchronize schematic symbols and pin assignments with physical footprints for U8 (QFN-64), D3 (SOT-23-6), J3 (USB-C 16-pin), U12 (QFN-20), and J1-J7 shield mounting pads
- Update netclasses in openmotorbridge_main.kicad_pro (Power_12V, Power_5V_3V3, USB_Diff_90)
- Update 3D renders and layout export diagrams in docs/images/pcba/
Parts:
- removed ANT2: Taoglas_FXUWB10_6.5GHz_Ch5_Floor, U.FL_Hirose_U.FL-R-SMT-1_Vertical, symbol OMB_Main:ANT2_Taoglas_FXUWB10_6.5GHz_Ch5_Floor
- removed J1: DEUTSCH_DTM12_IDC_HEADER, Connector_IDC:IDC-Header_2x06_P2.54mm_Vertical, symbol OMB_Main:J1_DEUTSCH_DTM12_IDC_HEADER
- removed J3: USB2_IDC_HEADER_9PIN, Connector_IDC:IDC-Header_2x05_P2.54mm_Vertical, symbol OMB_Main:J3_USB2_IDC_HEADER_9PIN
- removed U8: DW3110, QFN-16-1EP_3x3mm_P0.5mm_EP1.7x1.7mm_ThermalVias, symbol OMB_Main:U8_DW3110
- removed Y1_UWB: 38.4MHz, Crystal:Crystal_SMD_2016-4Pin_2.0x1.6mm, symbol OMB_Main:Y1_UWB_38.4MHz
- added C5: 100nF_ESP_EN, Capacitor_SMD:C_0603_1608Metric, symbol OMB_Main:C_100nF_0603
- added D3: LM66100_Ideal_Diode, Package_TO_SOT_SMD:SOT-23-6, symbol OMB_Main:D_OR_IDEAL_DIODE
- added J1: MicroLock_Plus_6Pin_Vertical, Connector_Molex:Molex_Micro-Lock_Plus_505568-0671_1x06_P1.25mm_Vertical, symbol OMB_Main:J_PWR_CAN_6PIN
- added J3: USB_C_Service_Port, Connector_USB:USB_C_Receptacle_HRO_TYPE-C-31-M-12_16P, symbol OMB_Main:J_USBC_16PIN
- added J6: Picoflex_16Pin_2x08_Vertical, Connector_Molex:Molex_Picoflex_90814-0016_2x08_P1.27mm_Vertical, symbol OMB_Main:J_PERIPH_16PIN
- added J7: USB_Reserve_Port7, Connector_Molex:Molex_Micro-Lock_Plus_505568-0471_1x04_P1.25mm_Vertical, symbol OMB_Main:J_RES_4PIN
- added R12: 100k_BAT_TOP, Resistor_SMD:R_0603_1608Metric, symbol OMB_Main:R_100k_0603
- added R13: 100k_BAT_BOT, Resistor_SMD:R_0603_1608Metric, symbol OMB_Main:R_100k_0603
- added R14: 10k_BAT_NTC, Resistor_SMD:R_0603_1608Metric, symbol OMB_Main:R_10k_0603
- added R3: 5k1_CC1, Resistor_SMD:R_0603_1608Metric, symbol OMB_Main:R_5k1_0603
- added R4: 5k1_CC2, Resistor_SMD:R_0603_1608Metric, symbol OMB_Main:R_5k1_0603
- added R5: 10k_HUB_RST, Resistor_SMD:R_0603_1608Metric, symbol OMB_Main:R_10k_0603
- added R6: 10k_ESP_EN, Resistor_SMD:R_0603_1608Metric, symbol OMB_Main:R_10k_0603
- added R7: 100k_KL15_TOP, Resistor_SMD:R_0603_1608Metric, symbol OMB_Main:R_100k_0603
- added R8: 22k_KL15_BOT, Resistor_SMD:R_0603_1608Metric, symbol OMB_Main:R_22k_0603
- added U12: TPS25921_Quad_eFuse, Package_DFN_QFN:QFN-20-1EP_3.5x4mm_P0.5mm, symbol OMB_Main:U12_QUAD_EFUSE
- added U8: USB2517I-JZX, Package_DFN_QFN:QFN-64-1EP_9x9mm_P0.5mm_EP7.15x7.15mm, symbol OMB_Main:U_HUB_USB2517I
- added Y2: 24.000MHz, Crystal:Crystal_SMD_2016-4Pin_2.0x1.6mm, symbol OMB_Main:Y2_HUB_24MHz
- J4: footprint Connector_JST:JST_PH_B3B-PH-K_1x03_P2.00mm_Vertical -> Connector_Molex:Molex_Micro-Lock_Plus_505568-0371_1x03_P1.25mm_Vertical
- J5: footprint Connector_JST:JST_PH_B4B-PH-K_1x04_P2.00mm_Vertical -> Connector_Molex:Molex_Micro-Lock_Plus_505568-0471_1x04_P1.25mm_Vertical
- U2: value ESP32-S3-WROOM-1U-N16R8 -> ESP32-S31-WROOM-1U; symbol OMB_Main:U2_ESP32-S3-WROOM-1U-N16R8 -> OMB_Main:U2_ESP32-S31-WROOM-1U
Connections:
- net CAN_H: now also J1.4
- net CAN_L: now also J1.5
- net ESP_EN: now also C5.1, R6.1
- net GND_PWR: now also J4.MP1, J4.MP2, J5.MP1, J5.MP2, C5.2, D3.2 (GND1), D3.5 (GND2), J1.3, J1.MP1, J1.MP2, J3.A1, J3.A12, J6.10, J6.14, J6.2, J6.6, J6.MP1, J6.MP2, J7.4, J7.MP1, J7.MP2, R13.2, R3.2, R4.2, R8.2, U12.10 (GND), U12.EP, U8.10 (GND), U8.11 (GND), U8.12 (GND), U8.13 (GND), U8.14 (GND), U8.15 (GND), U8.18 (GND), U8.19 (GND), U8.20 (GND), U8.21 (GND), U8.22 (GND), U8.23 (GND), U8.26 (GND), U8.27 (GND), U8.28 (GND), U8.29 (GND), U8.3 (GND), U8.30 (GND), U8.31 (GND), U8.50 (GND), U8.51 (GND), U8.52 (GND), U8.53 (GND), U8.54 (GND), U8.55 (GND), U8.58 (GND), U8.59 (GND), U8.6 (GND), U8.62 (GND), U8.63 (GND), U8.64 (GND), U8.7 (GND), U8.EP, Y2.2, Y2.4; no longer J5.3
- net GND_SHIELD: now also J1.6, J3.SH1, J3.SH2
- net KL30_IN: now also J1.1, U12.1 (VIN1), U12.2 (VIN2); no longer J5.1
- net VCC_3V3: now also R14.2, R5.2, R6.2, U8.1 (VDD33), U8.34 (VDD33), U8.35 (VDD33), U8.36 (VDD33), U8.37 (VDD33), U8.38 (VDD33), U8.39 (VDD33), U8.42 (VDD33), U8.43 (VDD33), U8.44 (VDD33), U8.45 (VDD33), U8.46 (VDD33), U8.47 (VDD33)
- net VCC_5V: now also D3.3 (VOUT1), D3.4 (VOUT2), J7.1
- net KL15_SENSE: now reaches U2.5
- net KL15_SENSE: now also R7.2, R8.1
- net USB_D_N renamed ESP_USB_DM
- net ESP_USB_DM: now also U8.16 (ESP_DM)
- net USB_D_P renamed ESP_USB_DP
- net ESP_USB_DP: now also U8.17 (ESP_DP)
- net UWB_CS renamed BAT_NTC
- net BAT_NTC: now also J5.3, R14.1
- net UWB_IRQ renamed BAT_SENSE
- net BAT_SENSE: now also R12.2, R13.1
- new net BAT_PLUS: J5.1, R12.1
- new net BT_USB_DM: U8.56 (BT_DM), U9.13
- new net BT_USB_DP: U8.57 (BT_DP), U9.14
- new net BUS1_DM: J6.3, U8.24 (BUS1_DM)
- new net BUS1_DP: J6.4, U8.25 (BUS1_DP)
- new net BUS2_DM: J6.7, U8.32 (BUS2_DM)
- new net BUS2_DP: J6.8, U8.33 (BUS2_DP)
- new net BUS3_DM: J6.11, U8.40 (BUS3_DM)
- new net BUS3_DP: J6.12, U8.41 (BUS3_DP)
- new net BUS4_DM: J6.15, U8.48 (BUS4_DM)
- new net BUS4_DP: J6.16, U8.49 (BUS4_DP)
- new net CC1: J3.A5, R3.1
- new net CC2: J3.A8, R4.1
- new net HUB_RESET_N: R5.1, U8.2 (RESET_N)
- new net KL15_IN: J1.2, R7.1
- new net RES_USB_DM: J7.2, U8.60 (RES_DM)
- new net RES_USB_DP: J7.3, U8.61 (RES_DP)
- new net USBC_DM: J3.A7, U8.8 (USBC_DM)
- new net USBC_DP: J3.A6, U8.9 (USBC_DP)
- new net USBC_VBUS: D3.1 (VIN1), D3.6 (VIN2), J3.A4, J3.A9
- new net VBUS_FRONT: J6.1, U12.5 (OUT1)
- new net VBUS_POD1: J6.5, U12.6 (OUT2)
- new net VBUS_POD2: J6.9, U12.7 (OUT3)
- new net VBUS_RADAR: J6.13, U12.8 (OUT4)
- new net XTALIN_24M: U8.4 (XTALIN), Y2.1
- new net XTALOUT_24M: U8.5 (XTALOUT), Y2.3
- no-connect marks 0 -> 24
Other:
- title: OpenMotorBridge v9.6 - Zentralbox Central Unit (PCBA 01) -> OpenMotorBridge v10.0 - Zentralbox Central Unit (PCBA 01)
