File: hardware/kicad_omm446_intercom/openmotorbridge_omm446_intercom.kicad_pcb (KiCad board)
At the start: 4 copper layers, 60 x 30 mm, 22 parts, among them J1 TYPE-C-31-M-12_IP67, SW1 BTN_PTT, SW2 BTN_MODE, SW3 BTN_CH_UP, SW4 BTN_CH_DOWN, U1 ESP32-C6-MINI-1U, U2 BQ24075RGTR, U3 SA818-DMR, U4 ES8388, U5 ME6211C33M5G, U6 ESP32-PICO-V3-02

Commit message: feat(hw): finalize PCB lineup routing, sync PCBA 03 cartridge with J_PROG header and DTM12 schematics
- PCBA 01 (Central Box): Remediate net routing, DTM12 hierarchical schematic synchronization, 100% routed, 0 DRC errors.
- PCBA 03 (Smart Modular Cartridge): Position and route J_PROG 4-pin SMD programming header on F.Cu at (108.0, 89.61), synchronize CPL and schematic, 100% routed, 0 DRC errors.
- PCBA 05 (Universal Front Node): Preconnect and routing verified, 100% routed, 0 DRC errors.
- PCBA 07 (LoRa Smart-Keyfob): Routing and DRC verified, 100% routed, 0 DRC errors.
- PCBA 08 (Radar 2.0 Sub-MCU & Wings): Sub-MCU routing and HF isolation verified, 100% routed, 0 DRC errors.
- PCBA 10 (OMM 446 PMR/DMR Intercom): KiCad DRC verified, 100% routed, 0 DRC errors.
- Firmware: Align configuration headers across front_node and smart_cartridge.
- Tools: Add comprehensive preflight PCBA audit suite tools/audit_pcbas_preflight.py.
Routing:
- net GND: track 25.2 -> 24.1 mm
