File: hardware/kicad_omm446_intercom/openmotorbridge_omm446_intercom.kicad_sch (KiCad schematic)
At the start: 16 parts, among them J1 TYPE-C-31-M-12_IP67, J2 BM08B-SRSS-TB, SW1 BTN_PTT, SW2 BTN_MODE, SW3 BTN_CH_UP, SW4 BTN_CH_DOWN, U1 ESP32-C6-MINI-1U, U2 BQ24075RGTR, U3 SA818-DMR, U4 ES8388, U5 ME6211C33M5G

Commit message: feat(hw): finalize PCBA 10 OMM 446 routing, schematic parity, 3D renders, and JLCPCB packages
Parts:
- removed J2: BM08B-SRSS-TB, Connector_JST:JST_SH_BM08B-SRSS-TB_1x08-1MP_P1.00mm_Vertical, symbol Connector:JST_SH_8Pin_Kelvin
Changed lines of the file:
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@@
 		(pin "B5")
 		(pin "B8")
+		(pin "SH")
 	)
 	(symbol (lib_id "Power:USBLC6-2SC6") (at 60.0 140.0 0) (unit 1)
@@
 		(pin "17")
 		(pin "18")
-	)
-	(symbol (lib_id "Connector:JST_SH_8Pin_Kelvin") (at 60.0 180.0 0) (unit 1)
-		(in_bom yes) (on_board yes) (dnp no)
-		(property "Reference" "J2" (at 60.0 165.0 0) (effects (font (size 1.27 1.27))))
-		(property "Value" "BM08B-SRSS-TB" (at 60.0 168.0 0) (effects (font (size 1.27 1.27))))
-		(property "Footprint" "Connector_JST:JST_SH_BM08B-SRSS-TB_1x08-1MP_P1.00mm_Vertical" (at 0 0 0) (effects (font (size 1.27 1.27)) hide))
-		(pin "1")
-		(pin "2")
-		(pin "3")
-		(pin "4")
-		(pin "5")
-		(pin "6")
-		(pin "7")
-		(pin "8")
 	)
 	(symbol (lib_id "MCU:ESP32-C6-MINI-1U") (at 80.0 140.0 0) (unit 1)
@@
 		(pin "1")
 		(pin "2")
+		(pin "3")
 	)
 	(symbol (lib_id "Connector:Battery_JST_2Pin") (at 240.0 260.0 0) (unit 1)
@@
 		(pin "1")
 		(pin "2")
+		(pin "MP")
 	)
 	(symbol (lib_id "Pad:Contact_Spring") (at 280.0 260.0 0) (unit 1)

Commit message: feat(hw,docs): implement Dual-Engine OMB Lite architecture for PCBA 09 and PCBA 10
- Schematic: Add ESP32-PICO-V3-02 (BT Classic/BLE co-processor) and Johanson 2450AT18 chip antenna
- PCB: Add Grobplatzierung and Vorverbindung nets on B.Cu for PCBA 09 and PCBA 10
- Firmware: Add co-processor UART link config and disable BT on C6 to eliminate CoEx time-slicing
- Documentation: Add Dual-Engine architecture, Cardo DMC Bridge / Sena Bridge, and Profile C OMB Lite
Parts:
- added ANT1: 2.45GHz_Chip_Antenna, RF_Antenna:Johanson_2450AT18x100, symbol RF_Antenna:Johanson_2450AT18x100
- added U6: ESP32-PICO-V3-02, Package_DFN_QFN:QFN-48-1EP_7x7mm_P0.5mm_EP5.3x5.3mm, symbol MCU:ESP32-PICO-V3-02
Changed lines of the file:
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@@
 		(rev "v2.0-dmr-pmr446")
 		(company "OpenMotorBridge Open Source Hardware")
-		(comment 1 "ESP32-C6-MINI-1U (U.FL), NiceRF SA818-DMR (CMX7141 + PA), ES8388 Stereo Codec, BQ24075 PMIC")
+		(comment 1 "Dual-Engine: ESP32-C6 (PMR/DMR Controller) + ESP32-PICO-V3-02 (BT Classic/BLE Bridge), NiceRF SA818-DMR, ES8388")
 		(comment 2 "Dual-Mode: 16CH PMR446 Analog FM & DMR Tier I Digital. Dual-Power: 0.2W Helmet / 0.5W Bike")
 	)
@@
 	(global_label "BTN_CH_UP" (shape input) (at 200.0 95.0 180) (effects (font (size 1.27 1.27)) (justify right)))
 	(global_label "BTN_CH_DOWN" (shape input) (at 200.0 100.0 180) (effects (font (size 1.27 1.27)) (justify right)))
+	(global_label "BT_UART_TX" (shape output) (at 260.0 30.0 0) (effects (font (size 1.27 1.27)) (justify left)))
+	(global_label "BT_UART_RX" (shape input) (at 260.0 35.0 180) (effects (font (size 1.27 1.27)) (justify right)))
+	(global_label "BT_UART_RTS" (shape output) (at 260.0 40.0 0) (effects (font (size 1.27 1.27)) (justify left)))
+	(global_label "BT_UART_CTS" (shape input) (at 260.0 45.0 180) (effects (font (size 1.27 1.27)) (justify right)))
+	(global_label "BT_RESET" (shape output) (at 260.0 50.0 0) (effects (font (size 1.27 1.27)) (justify left)))
+	(global_label "BT_BOOT" (shape output) (at 260.0 55.0 0) (effects (font (size 1.27 1.27)) (justify left)))
+	(global_label "BT_ANT" (shape bidirectional) (at 260.0 60.0 0) (effects (font (size 1.27 1.27)) (justify left)))
 	(symbol (lib_id "Audio:ES8388") (at 120.0 100.0 0) (unit 1)
 		(in_bom yes) (on_board yes) (dnp no)
@@
 		(pin "1")
 	)
+	(symbol (lib_id "MCU:ESP32-PICO-V3-02") (at 200.0 140.0 0) (unit 1)
+		(in_bom yes) (on_board yes) (dnp no)
+		(property "Reference" "U6" (at 200.0 110.0 0) (effects (font (size 1.27 1.27))))
+		(property "Value" "ESP32-PICO-V3-02" (at 200.0 113.0 0) (effects (font (size 1.27 1.27))))
+		(property "Footprint" "Package_DFN_QFN:QFN-48-1EP_7x7mm_P0.5mm_EP5.3x5.3mm" (at 0 0 0) (effects (font (size 1.27 1.27)) hide))
+		(property "LCSC" "C2686884" (at 0 0 0) (effects (font (size 1.27 1.27)) hide))
+		(pin "1")
+		(pin "2")
+		(pin "3")
+		(pin "4")
+		(pin "9")
+		(pin "19")
+		(pin "20")
+		(pin "21")
+		(pin "23")
+		(pin "37")
+		(pin "40")
+		(pin "41")
+		(pin "43")
+		(pin "46")
+		(pin "49")
+	)
+	(symbol (lib_id "RF_Antenna:Johanson_2450AT18x100") (at 250.0 140.0 0) (unit 1)
+		(in_bom yes) (on_board yes) (dnp no)
+		(property "Reference" "ANT1" (at 250.0 130.0 0) (effects (font (size 1.27 1.27))))
+		(property "Value" "2.45GHz_Chip_Antenna" (at 250.0 133.0 0) (effects (font (size 1.27 1.27))))
+		(property "Footprint" "RF_Antenna:Johanson_2450AT18x100" (at 0 0 0) (effects (font (size 1.27 1.27)) hide))
+		(property "LCSC" "C2909988" (at 0 0 0) (effects (font (size 1.27 1.27)) hide))
+		(pin "1")
+		(pin "2")
+	)
 )

Commit message: feat(omm): set compact stubby antenna as helmet default, add internal J_HELMET audio & maintain external USB-C
Parts:
- J_HELMET: renamed from PAD1; value Contact_Spring_Helix -> HELMET_AUDIO_6P; footprint TestPoint:TestPoint_Pad_D3.0mm -> Connector_JST:JST_SH_SM06B-SRSS-TB_1x06-1MP_P1.00mm_Horizontal; symbol Pad:Contact_Spring -> Connector:Conn_01x06_Pin; LCSC (none) -> C136657
Changed lines of the file:
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@@
 		(pin "MP")
 	)
-	(symbol (lib_id "Pad:Contact_Spring") (at 280.0 260.0 0) (unit 1)
+	(symbol (lib_id "Connector:Conn_01x06_Pin") (at 280.0 260.0 0) (unit 1)
 		(in_bom yes) (on_board yes) (dnp no)
-		(property "Reference" "PAD1" (at 280.0 245.0 0) (effects (font (size 1.27 1.27))))
-		(property "Value" "Contact_Spring_Helix" (at 280.0 248.0 0) (effects (font (size 1.27 1.27))))
-		(property "Footprint" "TestPoint:TestPoint_Pad_D3.0mm" (at 0 0 0) (effects (font (size 1.27 1.27)) hide))
+		(property "Reference" "J_HELMET" (at 280.0 245.0 0) (effects (font (size 1.27 1.27))))
+		(property "Value" "HELMET_AUDIO_6P" (at 280.0 248.0 0) (effects (font (size 1.27 1.27))))
+		(property "Footprint" "Connector_JST:JST_SH_SM06B-SRSS-TB_1x06-1MP_P1.00mm_Horizontal" (at 0 0 0) (effects (font (size 1.27 1.27)) hide))
+		(property "LCSC" "C136657" (at 0 0 0) (effects (font (size 1.27 1.27)) hide))
 		(pin "1")
+		(pin "2")
+		(pin "3")
+		(pin "4")
+		(pin "5")
+		(pin "6")
 	)
 	(symbol (lib_id "MCU:ESP32-PICO-V3-02") (at 200.0 140.0 0) (unit 1)

Commit message: fix(hardware): fleet-wide 7-PCBA remediation, schematic parity & doc alignment
- PCBA 01 (Central Box): Synchronized DTM-12 schematic and PCB routing, purged obsolete analog audio transformers/HD26 connector.
- PCBA 03 (Smart Cartridge): Verified Kelvin ground isolation on J_AUDIO_PWR, resolved U1.16 BAY_SELECT single net.
- PCBA 05 (Front Node): Mapped DW3110 UWB SPI/IRQ/RST to ESP32-S3 pads 30-35, connected MK1 I2S MEMS mic and Y_UWB crystal.
- PCBA 07 (Smart Keyfob): Connected 12 unrouted signals (SX1262 LoRa SPI, DRV2605L I2C, SWD, RTC crystal, buttons) to nRF52840 pads.
- PCBA 08 (Radar Sub-MCU): Synchronized J1.1 power rail to VCC_5V, connected Y1_UWB crystal to DW3110 pads 4 & 5.
- PCBA 09 & PCBA 10 (OMM 2.4 GHz & 446 MHz): Verified 4-layer stackup, BQ24075 ground ties, SA818 isolation, and vertical B.Cu J_HELMET orientation.
- Tools: Added verify_hardware_integrity.py with automated DRC/parity/single-net/floating-pad checks (all 7 PCBAs HEALTHY).
- Docs: Synchronized docs/de and docs/en hardware specifications, pinouts, and DTM-12 architecture.
Parts:
- added H1, H2, H3, H4: M2_MountingHole, MountingHole_2.2mm_M2_Pad, symbol Mechanical:MountingHole_Pad
- BAT1: value BM02B-SRSS-TB -> JST_2P_LiPo_600mAh; footprint Connector_JST:JST_SH_BM02B-SRSS-TB_1x02-1MP_P1.00mm_Vertical -> JST_SH_BM02B-SRSS-TB_1x02-1MP_P1.00mm_Vertical
- D1: footprint LED_SMD:LED_WS2812B-2020_PLCC4_2.0x2.0mm -> LED_WS2812B-2020_PLCC4_2.0x2.0mm
- D2: footprint Package_TO_SOT_SMD:SOT-23-6 -> SOT-23-6
- J1: footprint Connector_USB:USB_C_Receptacle_HRO_TYPE-C-31-M-12 -> USB_C_Receptacle_HRO_TYPE-C-31-M-12
- J_HELMET: footprint Connector_JST:JST_SH_SM06B-SRSS-TB_1x06-1MP_P1.00mm_Horizontal -> JST_SH_BM06B-SRSS-TB_1x06-1MP_P1.00mm_Vertical; LCSC C136657 -> (none)
- J_RF: footprint Connector_Coaxial:U.FL_Hirose_U.FL-R-SMT-1_Vertical -> U.FL_Hirose_U.FL-R-SMT-1_Vertical
- SW1, SW2, SW3, SW4: footprint Button_Switch_SMD:SW_Push_SPST_NO_Alps_SKRK -> SW_Push_SPST_NO_Alps_SKRK
- U1: footprint RF_Module:ESP32-C6-MINI-1U -> ESP32-S2-MINI-1U
- U2: footprint Package_DFN_QFN:VQFN-16-1EP_3x3mm_P0.5mm_EP1.8x1.8mm -> VQFN-16-1EP_3x3mm_P0.5mm_EP1.8x1.8mm
- U3: footprint RF_Module:NiceRF_SA818-DMR_SMD_38x16mm -> NiceRF_SA818-DMR_SMD_38x16mm
- U4: footprint Package_DFN_QFN:QFN-28-1EP_4x4mm_P0.4mm_EP2.4x2.4mm -> QFN-28-1EP_4x4mm_P0.4mm_EP2.4x2.4mm
- U5: footprint Package_TO_SOT_SMD:SOT-23-5 -> SOT-23
Connections:
- net AGND: now also U3.18 (AGND), U4.16 (AGND), U4.17 (VREF), U4.18 (MICBIAS)
- net AGND_MIC: now also J_HELMET.5 (Pin_5), U4.20 (MIC1N)
- net AGND_SPK: now also J_HELMET.3 (Pin_3), U4.24 (PGND)
- net BT_ANT: now also ANT1.1 (FEED), U6.2 (LNA_IN)
- net BT_BOOT: now also U1.12 (IO10), U6.23 (IO0_BOOT)
- net BT_RESET: now also U1.13 (IO11), U6.9 (EN)
- net BT_UART_CTS: now also U1.26 (GND), U6.20 (IO13_CTS)
- net BT_UART_RTS: now also U1.27 (EP), U6.21 (IO15_RTS)
- net BT_UART_RX: now also U1.29 (IO1), U6.40 (U0RXD)
- net BT_UART_TX: now also U1.28 (IO0), U6.41 (U0TXD)
- net CHG_STAT: now also U1.7 (IO7), U2.9 (~CHG)
- net GND: now also ANT1.2 (GND), BAT1.2 (-), BAT1.MP, D1.1 (DO), D1.3 (VDD), D2.2 (GND), J1.A5 (HP_OUT_L), J1.B5 (HP_OUT_R), J_HELMET.MP, J_RF.2 (Ext), J_RF.3 (Ext), SW1.2, SW2.2, SW3.2, SW4.2, U1.1 (GND), U1.3 (EN), U1.40 (GND), U1.41 (GND), U1.42 (GND), U1.43 (GND), U1.44 (GND), U1.45 (GND), U1.46 (GND), U1.47 (GND), U1.48 (GND), U1.49 (GND), U1.50 (GND), U1.51 (GND), U1.52 (GND), U1.53 (GND), U1.54 (GND), U1.55 (GND), U1.56 (GND), U1.57 (GND), U1.58 (GND), U1.59 (GND), U1.60 (GND), U1.61 (GND), U1.62 (GND), U1.63 (GND), U1.64 (GND), U1.65 (GND), U2.1 (TS), U2.12 (ILIM), U2.14 (TMR), U2.15 (ISET), U2.16 (SYSOFF), U2.17 (EP), U2.4 (~CE), U2.5 (EN2), U2.6 (EN1), U2.7 (~PGOOD), U2.8 (VSS), U3.10 (RF_GND), U4.10 (DGND), U4.29 (EP), U4.8 (AD0), U5.1 (GND), U6.49 (GND), H1.1, H2.1, H3.1, H4.1
- net I2C_SCL: now also U1.11 (IO9), U4.7 (SCL)
- net I2C_SDA: now also U1.10 (IO8), U4.6 (SDA)
- net I2S_BCLK: now also U1.22 (IO20), U4.2 (BCLK)
- net I2S_DIN: now also U1.25 (IO23), U4.5 (SDOUT)
- net I2S_DOUT: now also U1.24 (IO22), U4.4 (SDIN)
- net I2S_MCLK: now also U1.21 (IO19), U4.1 (MCLK)
- net I2S_WS: now also U1.23 (IO21), U4.3 (WS)
- net PGND: now also J1.A1 (GND), J1.A12 (GND), J1.B1 (GND), J1.B12 (GND), J1.SH, U3.9 (PGND)
- net RF_ANT: now also J_RF.1 (In), U3.12 (ANT)
- net SA818_PTT: now also U1.18 (IO16), U3.5 (PTT)
- net SA818_PWR_HL: now also U1.20 (IO18), U3.7 (HL)
- net SA818_RXD: now also U1.17 (IO15), U3.16 (TXD)
- net SA818_SQL: now also U1.19 (IO17), U3.14 (SQ)
- net SA818_TXD: now also U1.16 (IO14), U3.15 (RXD)
- net SYS_PWR: now also U2.10 (OUT), U2.11 (OUT), U3.6 (PD), U3.8 (VBAT), U5.3 (VIN)
- net USB_DN: now also D2.3 (I/O2_IN), D2.4 (I/O2_OUT), J1.A7 (USB_DN), J1.B7 (USB_DN), U1.14 (IO12)
- net USB_DP: now also D2.1 (I/O1_IN), D2.6 (I/O1_OUT), J1.A6 (USB_DP), J1.B6 (USB_DP), U1.15 (IO13)
- net VBAT: now also BAT1.1 (+), U2.2 (BAT), U2.3 (BAT)
- net VBUS_5V: now also D2.5 (VBUS), J1.A4 (VBUS), J1.A9 (VBUS), J1.B4 (VBUS), J1.B9 (VBUS), U2.13 (IN)
- net VCC_3V3: now also D1.2 (DI), U1.2 (3V3), U3.1 (AUDIO_ON), U4.15 (AVDD), U4.23 (PVDD), U4.25 (CE), U4.9 (DVDD), U5.2 (VOUT), U6.1 (VDDA), U6.19 (VDD3P3_RTC), U6.3 (VDDA3P3), U6.37 (VDD3P3_CPU), U6.4 (VDDA3P3), U6.43 (VDDA), U6.46 (VDDA)
- net WS2812_DATA: now also D1.4 (GND), U1.6 (IO6)
- net AUDIO_OUT_R: now reaches U4.11 (ROUT1)
- net AUDIO_OUT_R: now also J_HELMET.2 (Pin_2)
- net AUDIO_OUT_L: now reaches U4.12 (LOUT1)
- net AUDIO_OUT_L: now also J_HELMET.1 (Pin_1)
- net VOICE_IN: now reaches U4.19 (MIC1P)
- net VOICE_IN: now also J_HELMET.4 (Pin_4)
- net SA818_MIC_IN: now reaches U3.17 (MIC_IN)
- net SA818_MIC_IN: now also U4.14 (LOUT2)
- net SA818_AF_OUT: now reaches U3.3 (AF_OUT)
- net SA818_AF_OUT: now also U4.21 (LIN2)
- net BTN_3: now reaches U1.4 (IO4)
- net BTN_3: now also SW3.1
- net BTN_4: now reaches U1.5 (IO5)
- net BTN_4: now also SW4.1
- net BTN_1: now reaches U1.8 (IO2)
- net BTN_1: now also J_HELMET.6 (Pin_6), SW1.1
- net BTN_2: now reaches U1.9 (IO3)
- net BTN_2: now also SW2.1
