File: hardware/kicad_smart_keyfob/openmotorbridge_smart_keyfob.kicad_sch (KiCad schematic)
At the start: 0 parts

Commit message: fix(keyfob): synchronize PCBA 07 schematic with PCB and pass prefab-gate check
Parts:
- added ANT1: 868MHz_CHIP_ANT, R_0805_2012Metric, symbol ANT1_sym
- added ANT2: 2.4GHz_BLE_ANT, R_0805_2012Metric, symbol ANT2_sym
- added C1: 10uF_VBAT, C_0603_1608Metric, symbol C1_sym
- added C2: 10uF_3V3, C_0603_1608Metric, symbol C2_sym
- added C3: 100nF_MCU, C_0402_1005Metric, symbol C3_sym
- added C4: 100nF_LORA, C_0402_1005Metric, symbol C4_sym
- added D1: WS2812B-2020, LED_WS2812B-2020_PLCC4_2.0x2.0mm, symbol D1_sym
- added J_QI: QI_COIL_ACH_2P, symbol J_QI_sym
- added J_SWD: SWD_PROG, PinHeader_1x04_P1.27mm_Vertical_SMD_Pin1Left, symbol J_SWD_sym
- added L1: 4.7uH_DCDC, L_0603_1608Metric, symbol L1_sym
- added LS1: CPT-9019S_BUZZER, Buzzer_CUI_CPT-9019S-SMT, symbol LS1_sym
- added M1: LRA_MOTOR_PADS, R_0805_2012Metric, symbol M1_sym
- added P_BAT: LIPO_BAT_PADS, R_0805_2012Metric, symbol P_BAT_sym
- added R1: 10k_PULLUP, R_0402_1005Metric, symbol R1_sym
- added R2: 10k_PULLUP, R_0402_1005Metric, symbol R2_sym
- added SW1: BTN_ARM, SW_Push_SPST_NO_Alps_SKRK, symbol SW1_sym
- added SW2: BTN_SOS, SW_Push_SPST_NO_Alps_SKRK, symbol SW2_sym
- added U1: nRF52840-QIAA, Nordic_AQFN-73-1EP_7x7mm_P0.5mm, symbol U1_sym
- added U2: SX1262IMLTRT, QFN-24-1EP_4x4mm_P0.5mm_EP2.8x2.8mm, symbol U2_sym
- added U3: DRV2605LDGSR, MSOP-10_3x3mm_P0.5mm, symbol U3_sym
- added U4: BQ51003YFPR, Texas_DSBGA-28_1.9x3mm_Layout4x7_P0.4mm, symbol U4_sym
- added U5: BQ25100YFPR, WSON-6-1EP_2x2mm_P0.65mm_EP1x1.6mm, symbol U5_sym
- added Y1: 32.000MHz, Crystal_SMD_2016-4Pin_2.0x1.6mm, symbol Y1_sym
- added Y2: 32.768kHz, Crystal_SMD_3215-2Pin_3.2x1.5mm, symbol Y2_sym
- added Y3: 32MHz_TCXO, Crystal_SMD_2016-4Pin_2.0x1.6mm, symbol Y3_sym
Connections:
- net BLE_ANT_50R: now also ANT2.1 (BLE_ANT_50R), U1.A8 (BLE_ANT_50R)
- net BTN_ARM_N: now also R1.2 (BTN_ARM_N), SW1.1 (BTN_ARM_N), U1.G1 (BTN_ARM_N)
- net BTN_SOS_N: now also R2.2 (BTN_SOS_N), SW2.1 (BTN_SOS_N), U1.J1 (BTN_SOS_N)
- net BUZZER_PWM: now also LS1.1 (BUZZER_PWM), U1.F2 (BUZZER_PWM)
- net CHG_STAT: now also U1.K2 (CHG_STAT), U5.4 (CHG_STAT)
- net DRV_EN: now also U1.M2 (DRV_EN), U3.1 (DRV_EN)
- net GND: now also ANT1.2 (GND), ANT2.2 (GND), C1.2 (GND), C2.2 (GND), C3.2 (GND), C4.2 (GND), D1.3 (GND), D1.4 (GND), J_SWD.4 (GND), LS1.2 (GND), P_BAT.2 (GND), SW1.2 (GND), SW2.2 (GND), U1.B11 (GND), U1.B9 (GND), U1.EP (GND), U2.10 (GND), U2.12 (GND), U2.17 (GND), U2.19 (GND), U2.2 (GND), U2.20 (GND), U2.21 (GND), U2.22 (GND), U2.23 (GND), U2.25 (GND), U2.3 (GND), U2.6 (GND), U3.4 (GND), U3.6 (GND), U3.8 (GND), U4.C1 (GND), U4.C2 (GND), U5.2 (GND), U5.5 (GND), U5.6 (GND), U5.7 (GND), Y1.2 (GND), Y1.4 (GND), Y3.2 (GND)
- net I2C_SCL: now also U1.P2 (I2C_SCL), U3.3 (I2C_SCL)
- net I2C_SDA: now also U1.N1 (I2C_SDA), U3.2 (I2C_SDA)
- net LED_DATA: now also D1.2 (LED_DATA), U1.L1 (LED_DATA)
- net LORA_ANT_50R: now also ANT1.1 (LORA_ANT_50R), U2.18 (LORA_ANT_50R)
- net LORA_BUSY: now also U1.W1 (LORA_BUSY), U2.8 (LORA_BUSY)
- net LORA_DIO1: now also U1.D2 (LORA_DIO1), U2.9 (LORA_DIO1)
- net LORA_MISO: now also U1.U1 (LORA_MISO), U2.16 (LORA_MISO)
- net LORA_MOSI: now also U1.T2 (LORA_MOSI), U2.15 (LORA_MOSI)
- net LORA_NSS: now also U1.R1 (LORA_NSS), U2.13 (LORA_NSS)
- net LORA_RESET: now also U1.Y2 (LORA_RESET), U2.7 (LORA_RESET)
- net LORA_SCK: now also U1.C1 (LORA_SCK), U2.14 (LORA_SCK)
- net LRA_NEG: now also M1.2 (LRA_NEG), U3.9 (LRA_NEG)
- net LRA_POS: now also M1.1 (LRA_POS), U3.7 (LRA_POS)
- net QI_AC1: now also J_QI.1 (QI_AC1), U4.A1 (QI_AC1), U4.A2 (QI_AC1)
- net QI_AC2: now also J_QI.2 (QI_AC2), U4.B1 (QI_AC2), U4.B2 (QI_AC2)
- net SWDCLK: now also J_SWD.3 (SWDCLK), U1.H2 (SWDCLK)
- net SWDIO: now also J_SWD.2 (SWDIO), U1.AC24 (SWDIO)
- net VBAT: now also C1.1 (VBAT), L1.2 (VBAT), P_BAT.1 (VBAT), U5.3 (VBAT)
- net VCC_3V3: now also C2.1 (VCC_3V3), C3.1 (VCC_3V3), C4.1 (VCC_3V3), D1.1 (VCC_3V3), J_SWD.1 (VCC_3V3), L1.1 (VCC_3V3), R1.1 (VCC_3V3), R2.1 (VCC_3V3), U1.B1 (VCC_3V3), U2.1 (VCC_3V3), U2.11 (VCC_3V3), U2.24 (VCC_3V3), U3.10 (VCC_3V3), U3.5 (VCC_3V3), Y3.4 (VCC_3V3)
- net VCC_QI_5V: now also U4.D1 (VCC_QI_5V), U4.D2 (VCC_QI_5V), U5.1 (VCC_QI_5V)
- new net RTC1: U1.F23 (RTC1), Y2.1 (RTC1)
- new net RTC2: U1.H23 (RTC2), Y2.2 (RTC2)
- new net TCXO_IN: U2.4 (TCXO_IN), Y3.1 (TCXO_IN)
- new net TCXO_OUT: U2.5 (TCXO_OUT), Y3.3 (TCXO_OUT)
- new net XTAL1: U1.A12 (XTAL1), Y1.1 (XTAL1)
- new net XTAL2: U1.A14 (XTAL2), Y1.3 (XTAL2)
Other:
- title: OpenMotorBridge 2-in-1 LoRa Smart-Keyfob & Pager (PCBA 07) -> OpenMotorBridge PCBA 07 - 2-in-1 LoRa Smart-Keyfob & Pager
