File: hardware/kicad_front_node/openmotorbridge_front_node.kicad_sch (KiCad schematic)
At the start: 58 parts, among them J1 12V_KL15_GND, J10 12V_QI_POWER, J11 12V_AUX_LIGHT, J12 QWIIC_I2C, J2 CAN_H_L_GND, J3 HANDLEBAR_MULTI_BTN, J4 USB_UPSTREAM_HOST, J5 USB_DN1_PHONE_PD20W, J5_MP3 USB_DN3_GLOVEBOX_PD20W, J6 USB_DN2_CP2AA_PIGTAIL, J6_AUX USB_DN4_COCKPIT_AUX, J7 USB-C_SERVICE, J8 ACTION_CAM_5V_PWR, J9 MIRROR_BSD_LEDS, K1 CPC1017N_CAN_RELAY, Q1 DMN63D8_BSD_MOSFET, Q2 TPS1H100_AUX_LIGHT, SW1 BOOT, SW2 RESET, U1 ESP32-S3-WROOM-1U, U2 USB2514Bi-AEZG, U3 TPS54302_5V_BUCK, U4 TPS2051B_PORT2_GATE, U5 SW3526_USB_PD1_20W, U6 TCAN334G_CAN, U7 TLV75533P_3V3_LDO, U8 SW3526_USB_PD3_20W, U9 DW3110, Y1 24.000MHz

Commit message: feat(front-node): finalize dual-satellite architecture, CAD enclosures and smart-screen mode
- PCBA 05: Streamline board to 44 components with J_COCKPIT (16-pin) & J_VEHICLE (8-pin) dual-row headers, ESP32-S3 and DW3000 UWB.
- Enclosure: Update 00_front_node_tub.scad with continuous O-ring perimeter groove and circular Ø 8.0 mm TPU cable gland entries.
- Satellites: Implement cockpit_breakout_block.scad (5x USB-C, PTT, M3 clamp, dovetail) and vehicle_breakout_block.scad (4x COTS latching sockets).
- Use-Cases: Document 3 cockpit operating modes for RKS/naked cruisers including Mode C standalone smart-screen (Carpuride/Chigee) on [HOST].
- CAD & BOM: Re-render all Front Node 3D previews, register build targets in build_cad_from_openscad.py, and update doc chapters 07, 08, 15 & bom_catalog.js.
Parts:
- removed C27: 10uF_50V_PD3, C_0805_2012Metric, symbol C27_sym
- removed C28: 22uF_25V_PD3, C_0805_2012Metric, symbol C28_sym
- removed J1: 12V_KL15_GND, JST_PH_B2B-PH-K_1x02_P2.00mm_Vertical, symbol J1_sym
- removed J10: 12V_QI_POWER, JST_PH_B2B-PH-K_1x02_P2.00mm_Vertical, symbol J10_sym
- removed J11: 12V_AUX_LIGHT, JST_PH_B2B-PH-K_1x02_P2.00mm_Vertical, symbol J11_sym
- removed J2: CAN_H_L_GND, JST_PH_B3B-PH-K_1x03_P2.00mm_Vertical, symbol J2_sym
- removed J3: HANDLEBAR_MULTI_BTN, JST_PH_B4B-PH-K_1x04_P2.00mm_Vertical, symbol J3_sym
- removed J4: USB_UPSTREAM_HOST, JST_PH_B4B-PH-K_1x04_P2.00mm_Vertical, symbol J4_sym
- removed J5: USB_DN1_PHONE_PD20W, JST_PH_B5B-PH-K_1x05_P2.00mm_Vertical, symbol J5_sym
- removed J5_MP3: USB_DN3_GLOVEBOX_PD20W, JST_PH_B5B-PH-K_1x05_P2.00mm_Vertical, symbol J5_MP3_sym
- removed J6: USB_DN2_CP2AA_PIGTAIL, JST_PH_B4B-PH-K_1x04_P2.00mm_Vertical, symbol J6_sym
- removed J6_AUX: USB_DN4_COCKPIT_AUX, JST_PH_B4B-PH-K_1x04_P2.00mm_Vertical, symbol J6_AUX_sym
- removed J8: ACTION_CAM_5V_PWR, JST_PH_B2B-PH-K_1x02_P2.00mm_Vertical, symbol J8_sym
- removed J9: MIRROR_BSD_LEDS, JST_PH_B3B-PH-K_1x03_P2.00mm_Vertical, symbol J9_sym
- removed L3: 4.7uH_PD3_Choke, L_Sunlord_MWSA0503S, symbol L3_sym
- removed U8: SW3526_USB_PD3_20W, QFN-28-1EP_4x4mm_P0.4mm_EP2.4x2.4mm_ThermalVias, symbol U8_sym
- added J_COCKPIT: COCKPIT_16P_SMD, PinHeader_2x08_P2.00mm_Vertical_SMD, symbol J_COCKPIT_sym
- added J_VEHICLE: VEHICLE_8P_SMD, PinHeader_2x04_P2.00mm_Vertical_SMD, symbol J_VEHICLE_sym
Connections:
- net +12V_AUX: now also J_VEHICLE.8 (+12V_AUX)
- net +12V_PROT: now also J_VEHICLE.5 (+12V_PROT)
- net BSD_LEFT_N: now also J_VEHICLE.6 (BSD_LEFT_N)
- net BSD_RIGHT_N: now also J_VEHICLE.7 (BSD_RIGHT_N)
- net CAN_H: now also J_VEHICLE.3 (CAN_H)
- net CAN_L: now also J_VEHICLE.4 (CAN_L)
- net GND: now also J_COCKPIT.13 (GND), J_COCKPIT.16 (GND), J_COCKPIT.4 (GND), J_COCKPIT.8 (GND), J_VEHICLE.2 (GND)
- net KL15_12V_SW: now also J_VEHICLE.1 (KL15_12V_SW)
- net PTT_IN1_N: now also J_COCKPIT.14 (PTT_IN1_N)
- net USB_DN1_CC: now also J_COCKPIT.12 (USB_DN1_CC)
- net USB_DN1_DM: now also J_COCKPIT.10 (USB_DN1_DM)
- net USB_DN1_DP: now also J_COCKPIT.11 (USB_DN1_DP)
- net USB_DN2_DM: now also J_COCKPIT.6 (USB_DN2_DM)
- net USB_DN2_DP: now also J_COCKPIT.7 (USB_DN2_DP)
- net USB_UP_DM: now also J_COCKPIT.2 (USB_UP_DM)
- net USB_UP_DP: now also J_COCKPIT.3 (USB_UP_DP)
- net USB_UP_VBUS: now also J_COCKPIT.1 (USB_UP_VBUS)
- net VBUS_PD1_OUT: now also J_COCKPIT.9 (VBUS_PD1_OUT)
- net VCC_5V: now also J_COCKPIT.15 (VCC_5V)
- net VCC_5V_OTTOCAST: now also J_COCKPIT.5 (VCC_5V_OTTOCAST)

Commit message: feat(front-node): integrate I2C bus into J_VEHICLE 12-pin, pass prefab-gate & update cad packages
Parts:
- removed J12: QWIIC_I2C, JST_SH_BM04B-SRSS-TB_1x04-1MP_P1.00mm_Vertical, symbol J12_sym
- H1, H2, H3, H4: now left out of the parts list
- J_VEHICLE: value VEHICLE_8P_SMD -> VEHICLE_12P_SMD; footprint PinHeader_2x04_P2.00mm_Vertical_SMD -> PinHeader_2x06_P2.00mm_Vertical_SMD
Connections:
- net GND: now also J_VEHICLE.10 (GND)
- net I2C_SCL: now also J_VEHICLE.12 (I2C_SCL)
- net I2C_SDA: now also J_VEHICLE.11 (I2C_SDA)
- net VCC_3V3: now also J_VEHICLE.9 (VCC_3V3)
