File: hardware/kicad_front_node/openmotorbridge_front_node.kicad_sch (KiCad schematic)
At the start: 43 parts, among them J7 USB-C_SERVICE, K1 CPC1017N_CAN_RELAY, Q1 DMN63D8_BSD_MOSFET, Q2 TPS1H100_AUX_LIGHT, SW1 BOOT, SW2 RESET, U1 ESP32-S3-WROOM-1U, U2 USB2514Bi-AEZG, U3 TPS54302_5V_BUCK, U4 TPS2051B_PORT2_GATE, U5 SW3526_USB_PD1_20W, U6 TCAN334G_CAN, U7 TLV75533P_3V3_LDO, U9 DW3110, Y1 24.000MHz

Commit message: feat(hw): update Front Node PCBA 05 to v10 ESP32-P4 + ESP32-E22 dual-chip architecture
- Replaced ESP32-S3 with ESP32-P4-NR16 (Dual-Core 400 MHz RISC-V, 0.0% radio on silicon, integrated 480 Mbps High-Speed USB 2.0 PHY)
- Added ESP32-E22-WROOM-2X2 companion radio (Wi-Fi 6E 5/6 GHz, 2x2 MIMO, dual U.FL ports ANT1/ANT2, connected via 4-bit SDIO 3.0)
- Eliminated 2.4 GHz radio completely from Front Node to avoid interference with Zentralbox QCC3084 / S31 Bluetooth / BLE mesh
- Removed legacy DW3110 UWB transceiver, UWB antenna, and old block pinheaders (J_VEHICLE 12P, J_COCKPIT 16P)
- Standardized all external connectors to automotive JST footprints (JST-GH, JST-SH, JST-PH) with clean unrouted layout ready for user routing
- Connected ESP32-P4 native USB HS to USB2514Bi Hub downstream port 4 for Harley Headset Emulation (MFi / UAC) and CDC-NCM Ethernet
- Routed independent USB-C service port directly to ESP32-P4 USB Serial/JTAG controller
- Updated 3D renders and documentation in docs/de/07_pcba_hardware_pinouts.md and docs/en/07_pcba_hardware_pinouts.md
Parts:
- removed ANT_UWB: Taoglas_FXUWB10, Connector_Coaxial:U.FL_Hirose_U.FL-R-SMT-1_Vertical, symbol ANT_UWB_sym
- removed D7: SS34_USB_OR, D_SMA, symbol D7_sym
- removed D8: SS34_BUCK_OR, D_SMA, symbol D8_sym
- removed J_COCKPIT: COCKPIT_16P_SMD, PinHeader_2x08_P2.00mm_Vertical_SMD, symbol J_COCKPIT_sym
- removed J_VEHICLE: VEHICLE_12P_SMD, PinHeader_2x06_P2.00mm_Vertical_SMD, symbol J_VEHICLE_sym
- removed MIC1: MSM261S4030H0R, InvenSense_ICS-43434-6_3.5x2.65mm, symbol MIC1_sym
- removed R8: 10k_FAULT, R_0603_1608Metric, symbol R8_sym
- removed Y_UWB: 38.4MHz, Crystal:Crystal_SMD_2016-4Pin_2.0x1.6mm, symbol Y_UWB_sym
- added ANT1: U.FL_5_6GHZ_MAIN, Connector_Coaxial:U.FL_Hirose_U.FL-R-SMT-1_Vertical, symbol ANT1_sym
- added ANT2: U.FL_5_6GHZ_MIMO, Connector_Coaxial:U.FL_Hirose_U.FL-R-SMT-1_Vertical, symbol ANT2_sym
- added J1: JST_GH_04P_BACKBONE, Connector_JST:JST_GH_SM04B-GHS-TB_1x04-1MP_P1.25mm_Horizontal, symbol J1_sym
- added J10: JST_PH_02P_NAVI_PWR, Connector_JST:JST_PH_S2B-PH-K_1x02_P2.00mm_Horizontal, symbol J10_sym
- added J4: JST_GH_06P_HUB_EXT, Connector_JST:JST_GH_SM06B-GHS-TB_1x06-1MP_P1.25mm_Horizontal, symbol J4_sym
- added J8: JST_PH_02P_CAM_PWR, Connector_JST:JST_PH_S2B-PH-K_1x02_P2.00mm_Horizontal, symbol J8_sym
- added J_AUX_LIGHT: JST_PH_02P_AUX_LIGHT, Connector_JST:JST_PH_S2B-PH-K_1x02_P2.00mm_Horizontal, symbol J_AUX_LIGHT_sym
- added J_CAN: JST_GH_02P_CAN, Connector_JST:JST_GH_SM02B-GHS-TB_1x02-1MP_P1.25mm_Horizontal, symbol J_CAN_sym
- added J_DISP_L: JST_SH_04P_DISP_L, Connector_JST:JST_SH_SM04B-SRSS-TB_1x04-1MP_P1.00mm_Horizontal, symbol J_DISP_L_sym
- added J_DISP_R: JST_SH_04P_DISP_R, Connector_JST:JST_SH_SM04B-SRSS-TB_1x04-1MP_P1.00mm_Horizontal, symbol J_DISP_R_sym
- added J_DONGLE: JST_GH_04P_DONGLE, Connector_JST:JST_GH_SM04B-GHS-TB_1x04-1MP_P1.25mm_Horizontal, symbol J_DONGLE_sym
- added J_POD_L: JST_GH_04P_POD_L, Connector_JST:JST_GH_SM04B-GHS-TB_1x04-1MP_P1.25mm_Horizontal, symbol J_POD_L_sym
- added J_POD_R: JST_GH_04P_POD_R, Connector_JST:JST_GH_SM04B-GHS-TB_1x04-1MP_P1.25mm_Horizontal, symbol J_POD_R_sym
- added J_SENSOR_EXT: JST_GH_06P_SENSOR_PUCK, Connector_JST:JST_GH_SM06B-GHS-TB_1x06-1MP_P1.25mm_Horizontal, symbol J_SENSOR_EXT_sym
- C_BUF: value 470uF_10V_POLYMER -> 470uF_25V_POLYMER
- H1, H2, H3, H4: now in the parts list
- J7: value USB-C_SERVICE -> USB_C_SERVICE
- U1: value ESP32-S3-WROOM-1U -> ESP32-P4-NR16
- U5: value SW3526_USB_PD1_20W -> SW3526_USB_PD1_30W
- U9: value DW3110 -> ESP32-E22-WROOM-2X2
Connections:
- net UWB_RF is gone; now on net GND: U9.15 (GND)
- net UWB_XTAL1 is gone; now on net SDIO_CLK: U9.4 (SDIO_CLK)
- net UWB_XTAL2 is gone; now on net SDIO_CMD: U9.5 (SDIO_CMD)
- net VBUS_BUCK_OUT is gone; now on net VCC_5V: L1.2 (VCC_5V)
- net VCC_5V_OTTOCAST is gone; now on net VCC_5V: U4.1 (VIN)
- net +12V_AUX: now also Q2.4 (OUT), J_AUX_LIGHT.1 (+12V_AUX); no longer Q2.6 (+12V_AUX), Q2.7 (+12V_AUX), Q2.8 (+12V_AUX)
- net +12V_PROT: now also C_BUF.1 (+12V_PROT), Q2.3 (VS), J10.1 (+12V_PROT); no longer D4.1 (+12V_PROT), Q2.11 (+12V_PROT), Q2.12 (+12V_PROT), Q2.13 (+12V_PROT), Q2.14 (+12V_PROT), Q2.15 (+12V_PROT), U5.2 (+12V_PROT), U5.28 (+12V_PROT)
- net CAN_H: now also K1.4 (DRAIN2), J_CAN.1 (CAN_H); no longer K1.3 (CAN_H)
- net CAN_L: now also J_CAN.2 (CAN_L)
- net CAN_SILENT: now also U6.5 (S); no longer U6.8 (CAN_SILENT)
- net CAN_TERM_R: now also K1.3 (DRAIN1); no longer K1.4 (CAN_TERM_R)
- net GND: now also LED1.1 (DO), LED1.4 (GND), MK1.4 (SELECT), Q2.5 (OUT_SENSE), U2.14 (GND), U5.4 (GND), U6.8 (NC), U9.13 (GND), U9.14 (GND), ANT1.2 (GND), ANT2.2 (GND), J1.2 (GND), J10.2 (GND), J4.2 (GND), J8.2 (GND), J_AUX_LIGHT.2 (GND), J_DISP_L.2 (GND), J_DISP_R.2 (GND), J_DONGLE.2 (GND), J_POD_L.4 (GND), J_POD_R.4 (GND), J_SENSOR_EXT.2 (GND); no longer J7.SH (GND), LED1.2 (GND), LED1.3 (GND), Q2.4 (GND), U1.40 (GND), U2.11 (GND), U2.25 (GND), U2.28 (GND), U2.34 (GND), U5.14 (GND), U5.29 (GND), U6.5 (GND), U9.1 (GND), U9.11 (GND), U9.3 (GND), U9.6 (GND)
- net HUB_RBIAS: now also U2.36 (RBIAS); no longer U2.35 (HUB_RBIAS)
- net I2C_SCL: now also J_DISP_L.3 (I2C_SCL), J_DISP_R.3 (I2C_SCL), J_SENSOR_EXT.4 (I2C_SCL)
- net I2C_SDA: now also J_DISP_L.4 (I2C_SDA), J_DISP_R.4 (I2C_SDA), J_SENSOR_EXT.3 (I2C_SDA)
- net MIC_I2S_DATA: now also J_SENSOR_EXT.5 (MIC_I2S_DATA)
- net MIC_I2S_WS: now also J_SENSOR_EXT.6 (MIC_I2S_WS)
- net SW_BUCK: now also U3.6 (BOOT)
- net SW_PD1_BUCK: now also U5.2 (SW); no longer U5.25 (SW_PD1_BUCK), U5.26 (SW_PD1_BUCK), U5.27 (SW_PD1_BUCK)
- net USB_DN1_DM: now also U5.8 (DM), J4.4 (USB_DN1_DM); no longer U5.17 (USB_DN1_DM)
- net USB_DN1_DP: now also U5.7 (DP), J4.3 (USB_DN1_DP); no longer U5.16 (USB_DN1_DP)
- net USB_DN2_DM: now also J_DONGLE.4 (USB_DN2_DM)
- net USB_DN2_DP: now also J_DONGLE.3 (USB_DN2_DP)
- net USB_DN3_DM: now also J4.6 (USB_DN3_DM)
- net USB_DN3_DP: now also J4.5 (USB_DN3_DP)
- net USB_SERV_DM: now also U1.24 (USB_SERV_DM); no longer U1.13 (USB_SERV_DM)
- net USB_SERV_DP: now also U1.25 (USB_SERV_DP); no longer U1.14 (USB_SERV_DP)
- net USB_UP_DM: now also U2.20 (USB_UP_DM), J1.4 (USB_UP_DM); no longer U2.30 (USB_UP_DM)
- net USB_UP_DP: now also U2.21 (USB_UP_DP), J1.3 (USB_UP_DP); no longer U2.31 (USB_UP_DP)
- net VBUS_PD1_OUT: now also U5.3 (VBUS), J4.1 (VBUS_PD1_OUT); no longer U5.21 (VBUS_PD1_OUT)
- net VCC_3V3: now also MK1.6 (VDD), U2.33 (RESET_N), U9.1 (VCC_3V3), J_DISP_L.1 (VCC_3V3), J_DISP_R.1 (VCC_3V3), J_SENSOR_EXT.1 (VCC_3V3); no longer MK1.4 (VCC_3V3), Q2.3 (VCC_3V3), U2.10 (VCC_3V3), U2.12 (VCC_3V3), U2.13 (VCC_3V3), U2.15 (VCC_3V3), U2.16 (VCC_3V3), U2.18 (VCC_3V3), U2.19 (VCC_3V3), U2.20 (VCC_3V3), U2.21 (VCC_3V3), U2.22 (VCC_3V3), U2.23 (VCC_3V3), U2.24 (VCC_3V3), U2.26 (VCC_3V3), U2.27 (VCC_3V3), U2.29 (VCC_3V3), U2.36 (VCC_3V3), U9.14 (VCC_3V3)
- net VCC_5V: now also LED1.3 (VDD), U2.24 (VBUS_DET), U3.4 (FB), J8.1 (VCC_5V), J_POD_L.1 (VCC_5V), J_POD_R.1 (VCC_5V); no longer C_BUF.1 (VCC_5V), LED1.1 (VCC_5V), U4.5 (VCC_5V)
- net WS2812B_DIN: now also LED1.2 (DI); no longer LED1.4 (WS2812B_DIN)
- net XTAL_IN: now also U2.12 (XTAL_IN); no longer U2.33 (XTAL_IN)
- net XTAL_OUT: now also U2.13 (XTAL_OUT); no longer U2.32 (XTAL_OUT)
- net USB_DN1_CC1: now reaches U5.5 (CC1)
- net USB_DN1_CC2: now reaches U5.6 (CC2)
- net E22_IRQ: now reaches U1.37 (E22_IRQ)
- net E22_IRQ: now also U9.10 (E22_IRQ)
- net BSD_LEFT_N renamed BSD_LED_L_N
- net BSD_LED_L_N: now also J_POD_L.2 (BSD_LED_L_N)
- net BSD_RIGHT_N renamed BSD_LED_R_N
- net BSD_LED_R_N: now also J_POD_R.2 (BSD_LED_R_N)
- net KL15_12V_SW renamed VIN_60W
- net VIN_60W: now also D4.1 (VIN_60W), J1.1 (VIN_60W)
- removed net OTTOCAST_FAULT_N: U1.38 (OTTOCAST_FAULT_N), U2.17 (OTTOCAST_FAULT_N), U4.3 (OTTOCAST_FAULT_N)
- net OTTOCAST_PWR_EN renamed CP2AA_FAULT_N
- net CP2AA_FAULT_N: now also U1.38 (CP2AA_FAULT_N); no longer U1.39 (OTTOCAST_PWR_EN)
- net PTT_IN1_N renamed BTN_SIG_L_N
- net BTN_SIG_L_N: now also J_POD_L.3 (BTN_SIG_L_N)
- net PTT_IN2_N renamed BTN_SIG_R_N
- net BTN_SIG_R_N: now also J_POD_R.3 (BTN_SIG_R_N)
- removed net PTT_IN3_N: U1.10 (PTT_IN3_N)
- removed net USB_DN1_CC: U5.18 (USB_DN1_CC), U5.19 (USB_DN1_CC)
- net USB_DN4_DM renamed USB_HS_DM
- net USB_HS_DM: now also U1.13 (USB_HS_DM)
- net USB_DN4_DP renamed USB_HS_DP
- net USB_HS_DP: now also U1.14 (USB_HS_DP)
- net UWB_CS renamed SDIO_D1
- net SDIO_D1: now also U9.7 (SDIO_D1); no longer U9.10 (UWB_CS)
- net UWB_IRQ renamed SDIO_D2
- net SDIO_D2: now also U9.8 (SDIO_D2); no longer U9.13 (UWB_IRQ)
- net UWB_MISO renamed SDIO_D0
- net SDIO_D0: now also U9.6 (SDIO_D0); no longer U9.8 (UWB_MISO)
- net UWB_MOSI renamed SDIO_CMD
- net SDIO_CMD: no longer U9.9 (UWB_MOSI)
- net UWB_RST renamed E22_RF_MIMO
- net E22_RF_MIMO: now also ANT2.1 (E22_RF_MIMO); no longer U1.35 (UWB_RST)
- net UWB_SCK renamed SDIO_CLK
- net SDIO_CLK: no longer U9.7 (UWB_SCK)
- new net CP2AA_PWR_EN: U1.39 (CP2AA_PWR_EN), U4.3 (EN)
- new net E22_EN: U1.40 (E22_EN), U9.3 (E22_EN)
- new net E22_RF_MAIN: ANT1.1 (E22_RF_MAIN), U9.11 (RF_MAIN)
- new net SDIO_D3: U1.35 (SDIO_D3), U9.9 (SDIO_D3)
- new net VCC_5V_DONGLE: J_DONGLE.1 (VCC_5V_DONGLE), U4.5 (VOUT)
Other:
- title: OpenMotorBridge Universal Front Node (Cockpit & Sensor Hub PCBA 05) -> OpenMotorBridge Universal Front Node (PCBA 05 v10.0)

Commit message: hardware(front-node): connect all nets in schematic and PCB with passives parity
Parts:
- removed J7: USB_C_SERVICE, USB_C_Receptacle_HRO_TYPE-C-31-M-12, symbol J7_sym
- removed J_CAN: JST_GH_02P_CAN, Connector_JST:JST_GH_SM02B-GHS-TB_1x02-1MP_P1.25mm_Horizontal, symbol J_CAN_sym
- removed K1: CPC1017N_CAN_RELAY, SOP-4_4.4x2.6mm_P1.27mm, symbol K1_sym
- removed R10: 120R_CAN, R_0603_1608Metric, symbol R10_sym
- removed R15: 5.1k_CC1, R_0603_1608Metric, symbol R15_sym
- removed R16: 5.1k_CC2, R_0603_1608Metric, symbol R16_sym
- removed U6: TCAN334G_CAN, SOIC-8_3.9x4.9mm_P1.27mm, symbol U6_sym
- added C_BOOT: 100nF_BOOT, C_0603_1608Metric, symbol C_BOOT_sym
- added C_EN: 1uF_EN, C_0603_1608Metric, symbol C_EN_sym
- added C_LED: 100nF_LED, C_0603_1608Metric, symbol C_LED_sym
- added C_MIC: 100nF_MIC, C_0603_1608Metric, symbol C_MIC_sym
- added C_VDD18: 1uF_1V8, C_0603_1608Metric, symbol C_VDD18_sym
- added C_XTAL1: 18pF, C_0603_1608Metric, symbol C_XTAL1_sym
- added C_XTAL2: 18pF, C_0603_1608Metric, symbol C_XTAL2_sym
- added R_BOOT: 10k_BOOT, R_0603_1608Metric, symbol R_BOOT_sym
- added R_BTN_L: 10k_PULLUP, R_0603_1608Metric, symbol R_BTN_L_sym
- added R_BTN_R: 10k_PULLUP, R_0603_1608Metric, symbol R_BTN_R_sym
- added R_E22_EN: 10k_E22_EN, R_0603_1608Metric, symbol R_E22_EN_sym
- added R_EN: 10k_EN, R_0603_1608Metric, symbol R_EN_sym
- added R_FB1: 100k_FB1, R_0603_1608Metric, symbol R_FB1_sym
- added R_FB2: 13.7k_FB2, R_0603_1608Metric, symbol R_FB2_sym
- added R_HUB_RST: 10k_HUB_RST, R_0603_1608Metric, symbol R_HUB_RST_sym
- added R_SCL: 4.7k_I2C, R_0603_1608Metric, symbol R_SCL_sym
- added R_SDA: 4.7k_I2C, R_0603_1608Metric, symbol R_SDA_sym
- added R_SDIO_CMD: 10k_PULLUP, R_0603_1608Metric, symbol R_SDIO_CMD_sym
- added R_SDIO_D0: 10k_PULLUP, R_0603_1608Metric, symbol R_SDIO_D0_sym
- added R_SDIO_D1: 10k_PULLUP, R_0603_1608Metric, symbol R_SDIO_D1_sym
- added R_SDIO_D2: 10k_PULLUP, R_0603_1608Metric, symbol R_SDIO_D2_sym
- added R_SDIO_D3: 10k_PULLUP, R_0603_1608Metric, symbol R_SDIO_D3_sym
Connections:
- net BTN_SIG_L_N: now also R_BTN_L.2 (BTN_L)
- net BTN_SIG_R_N: now also R_BTN_R.2 (BTN_R)
- net E22_EN: now also R_E22_EN.2 (E22_EN)
- net ESP_BOOT: now also R_BOOT.2 (ESP_BOOT)
- net ESP_EN: now also C_EN.1 (ESP_EN), R_EN.2 (ESP_EN)
- net GND: now also Q2.15 (EP_GND), U2.23 (CFG_SEL0), U2.25 (CFG_SEL1), U2.26 (NON_REM0), U2.27 (NON_REM1), U2.28 (TEST), U2.34 (GND), U5.29 (EP_GND), C_EN.2 (GND), C_LED.2 (GND), C_MIC.2 (GND), C_VDD18.2 (GND), C_XTAL1.2 (GND), C_XTAL2.2 (GND), R_FB2.2 (GND); no longer LED1.1 (DO), U7.4 (NC)
- net I2C_SCL: now also R_SCL.2 (I2C_SCL)
- net I2C_SDA: now also R_SDA.2 (I2C_SDA)
- net SDIO_CMD: now also R_SDIO_CMD.2 (SDIO_CMD)
- net SDIO_D0: now also R_SDIO_D0.2 (SDIO_D0)
- net SDIO_D1: now also R_SDIO_D1.2 (SDIO_D1)
- net SDIO_D2: now also R_SDIO_D2.2 (SDIO_D2)
- net SDIO_D3: now also R_SDIO_D3.2 (SDIO_D3)
- net SW_BUCK: now also C_BOOT.2 (SW); no longer U3.6 (BOOT)
- net VCC_3V3: now also U2.10 (PRTPWR1), U2.11 (OCS1_N), U2.15 (PRTPWR2), U2.16 (OCS2_N), U2.17 (PRTPWR3), U2.18 (OCS3_N), U2.19 (PRTPWR4), U2.22 (OCS4_N), U2.29 (VDD33), U2.30 (SCL), U2.32 (SDA), U2.35 (VDD33), C_MIC.1 (VDD), R_BOOT.1 (VCC_3V3), R_BTN_L.1 (VCC_3V3), R_BTN_R.1 (VCC_3V3), R_E22_EN.1 (VCC_3V3), R_EN.1 (VCC_3V3), R_HUB_RST.1 (VCC_3V3), R_SCL.1 (VCC_3V3), R_SDA.1 (VCC_3V3), R_SDIO_CMD.1 (VCC_3V3), R_SDIO_D0.1 (VCC_3V3), R_SDIO_D1.1 (VCC_3V3), R_SDIO_D2.1 (VCC_3V3), R_SDIO_D3.1 (VCC_3V3); no longer MK1.6 (VDD), U2.33 (RESET_N)
- net VCC_5V: now also C_LED.1 (VDD), R_FB1.1 (VCC_5V); no longer U3.4 (FB)
- net XTAL_IN: now also C_XTAL1.1 (XTAL_IN)
- net XTAL_OUT: now also C_XTAL2.1 (XTAL_OUT)
- removed net CAN_SILENT: U1.5 (CAN_SILENT)
- removed net CAN_TERM_EN: U1.15 (CAN_TERM_EN)
- removed net TWAI_RX: U1.36 (TWAI_RX)
- removed net TWAI_TX: U1.23 (TWAI_TX)
- removed net USB_SERV_DM: U1.24 (USB_SERV_DM)
- removed net USB_SERV_DP: U1.25 (USB_SERV_DP)
- new net BOOT_5V: C_BOOT.1 (BOOT), U3.6 (BOOT)
- new net FB_5V: R_FB1.2 (FB), R_FB2.1 (FB), U3.4 (FB)
- new net HUB_RESET_N: R_HUB_RST.2 (RESET_N), U2.33 (RESET_N)
- new net VDD18_CORE: C_VDD18.1 (VDD18), U2.31 (VDD18)
- no-connect marks 0 -> 2
Other:
- title: OpenMotorBridge Universal Front Node (PCBA 05 v10.0) -> OpenMotorBridge Universal Front Node (Cockpit & Sensor Hub PCBA 05 v10.0)

Commit message: feat(hardware): finalize Front Node PCBA 05 routing, net assignments, planes, and schematic parity
- Resolved all 0 unconnected items and cleared shorts on Front Node PCB
- Assigned nets across all 41 pins of U1, U5, Q2, LED1, and JST connectors
- Created and filled continuous GND and VCC_3V3 planes on In1.Cu and In2.Cu
- Synchronized KiCad schematic 1:1 to PCB achieving 0 blockers in prefab-gate check
- Removed obsolete CAN transceiver references from Front Node documentation
- Updated 3D renders for PCBA 05 top and bottom views in docs/images/pcba/
Parts:
- C24, C_BOOT, C_EN, C_LED, C_MIC, C_VDD18, C_XTAL1, C_XTAL2: footprint C_0603_1608Metric -> Capacitor_SMD:C_0603_1608Metric
- J1, J_DONGLE, J_POD_L, J_POD_R: footprint Connector_JST:JST_GH_SM04B-GHS-TB_1x04-1MP_P1.25mm_Horizontal -> JST_GH_SM04B-GHS-TB_1x04-1MP_P1.25mm_Horizontal
- J10, J8, J_AUX_LIGHT: footprint Connector_JST:JST_PH_S2B-PH-K_1x02_P2.00mm_Horizontal -> JST_PH_S2B-PH-K_1x02_P2.00mm_Horizontal
- J4, J_SENSOR_EXT: footprint Connector_JST:JST_GH_SM06B-GHS-TB_1x06-1MP_P1.25mm_Horizontal -> JST_GH_SM06B-GHS-TB_1x06-1MP_P1.25mm_Horizontal
- J_DISP_L, J_DISP_R: footprint Connector_JST:JST_SH_SM04B-SRSS-TB_1x04-1MP_P1.00mm_Horizontal -> JST_SH_SM04B-SRSS-TB_1x04-1MP_P1.00mm_Horizontal
- R5, R_BOOT, R_BTN_L, R_BTN_R, R_E22_EN, R_EN, R_FB1, R_FB2, R_HUB_RST, R_SCL, R_SDA, R_SDIO_CMD, R_SDIO_D0, R_SDIO_D1, R_SDIO_D2, R_SDIO_D3: footprint R_0603_1608Metric -> Resistor_SMD:R_0603_1608Metric
Connections:
- net +12V_AUX: now also Q2.10 (OUT), Q2.11 (OUT), Q2.12 (OUT), Q2.13 (OUT), Q2.14 (OUT), Q2.8 (OUT), Q2.9 (OUT)
- net +12V_PROT: now also Q2.6 (VS), Q2.7 (VS), U5.2 (VIN), U5.28 (VIN)
- net GND: now also J1.MP (SHIELD), J4.MP (SHIELD), J_DISP_L.MP (SHIELD), J_DISP_R.MP (SHIELD), J_DONGLE.MP (SHIELD), J_POD_L.MP (SHIELD), J_POD_R.MP (SHIELD), J_SENSOR_EXT.MP (SHIELD), U5.14 (GND), U7.4 (NC); no longer U5.4 (GND)
- net SW_PD1_BUCK: now also U5.25 (SW), U5.26 (SW), U5.27 (SW); no longer U5.2 (SW)
- net USB_DN1_CC1: now also U5.18 (CC1); no longer U5.5 (CC1)
- net USB_DN1_CC2: now also U5.19 (CC2); no longer U5.6 (CC2)
- net USB_DN1_DM: now also U5.17 (DM); no longer U5.8 (DM)
- net USB_DN1_DP: now also U5.16 (DP); no longer U5.7 (DP)
- net VBUS_PD1_OUT: now also U5.21 (VBUS); no longer U5.3 (VBUS)
- net LED1_DOUT: now reaches LED1.1 (DO)
- new net GPIO10: U1.10 (GPIO10)
- new net GPIO11: U1.11 (GPIO11)
- new net GPIO15: U1.15 (GPIO15)
- new net GPIO16: U1.16 (GPIO16)
- new net GPIO23: U1.23 (GPIO23)
- new net GPIO24: U1.24 (GPIO24)
- new net GPIO25: U1.25 (GPIO25)
- new net GPIO26: U1.26 (GPIO26)
- new net GPIO28: U1.28 (GPIO28)
- new net GPIO29: U1.29 (GPIO29)
- new net GPIO36: U1.36 (GPIO36)
- new net GPIO4: U1.4 (GPIO4)
- new net GPIO5: U1.5 (GPIO5)
- new net U5_BST: U5.3 (BST)
- new net U5_NC10: U5.10 (NC10)
- new net U5_NC11: U5.11 (NC11)
- new net U5_NC12: U5.12 (NC12)
- new net U5_NC13: U5.13 (NC13)
- new net U5_NC15: U5.15 (NC15)
- new net U5_NC20: U5.20 (NC20)
- new net U5_NC22: U5.22 (NC22)
- new net U5_NC23: U5.23 (NC23)
- new net U5_NC24: U5.24 (NC24)
- new net U5_NC5: U5.5 (NC5)
- new net U5_NC6: U5.6 (NC6)
- new net U5_NC7: U5.7 (NC7)
- new net U5_NC8: U5.8 (NC8)
- new net U5_NC9: U5.9 (NC9)
- new net U5_SW_SN: U5.4 (SW_SN)
- no-connect marks 2 -> 0
